File: RP_Led_Matrix.sch (KiCad schematic (older format))
At the start: 31 parts, among them J101 Conn_02x20_Odd_Even, Q101 2N3904, SW101 SW_Push_boxtec, SW102 SW_Push_boxtec, SW103 SW_Push_boxtec, SW104 SW_Push_boxtec, SW105 SW_Push_boxtec, SW106 SW_Push_boxtec, U101 ADS1015IDGS, U102 LM2595S-3.3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

Commit message: update Schema
-pwr flag eingefügt
-3.3V Analog Netzleibel eingefügt
Connections:
- net labels added: 3.3V_Analog
- wire segments 103 -> 110
Other:
- moved on the sheet: C106, FB101
Changed lines of the file:
@@
 	4750 1600 4750 1500
 Connection ~ 4350 1500
-Connection ~ 4750 1500
 Text Notes 1550 900  0    167  ~ 0
 Speisung 5V/3V3
@@
 L power:+5V #PWR0108
 U 1 1 5C770507
-P 2600 3500
-F 0 "#PWR0108" H 2600 3350 50  0001 C CNN
-F 1 "+5V" V 2615 3628 50  0000 L CNN
-F 2 "" H 2600 3500 50  0001 C CNN
-F 3 "" H 2600 3500 50  0001 C CNN
-	1    2600 3500
+P 3000 3500
+F 0 "#PWR0108" H 3000 3350 50  0001 C CNN
+F 1 "+5V" V 3015 3628 50  0000 L CNN
+F 2 "" H 3000 3500 50  0001 C CNN
+F 3 "" H 3000 3500 50  0001 C CNN
+	1    3000 3500
 	0    1    1    0
 $EndComp
@@
 	2600 3600 2500 3600
 Wire Wire Line
-	2600 3500 2500 3500
+	3000 3500 2900 3500
 Text Label 1750 3600 0    49   ~ 0
 SDA
@@
 L Device:Ferrite_Bead FB101
 U 1 1 5C77AF82
-P 5400 1500
-F 0 "FB101" V 5674 1500 50  0000 C CNN
-F 1 "Ferrite_Bead" V 5583 1500 50  0000 C CNN
-F 2 "" V 5330 1500 50  0001 C CNN
-F 3 "~" H 5400 1500 50  0001 C CNN
-	1    5400 1500
+P 6150 1500
+F 0 "FB101" V 6424 1500 50  0000 C CNN
+F 1 "Ferrite_Bead" V 6333 1500 50  0000 C CNN
+F 2 "" V 6080 1500 50  0001 C CNN
+F 3 "~" H 6150 1500 50  0001 C CNN
+	1    6150 1500
 	0    -1   -1   0
 $EndComp
@@
 L Device:C C106
 U 1 1 5C77B7BB
-P 5900 1750
-F 0 "C106" H 6015 1796 50  0000 L CNN
-F 1 "100n" H 6015 1705 50  0000 L CNN
-F 2 "" H 5938 1600 50  0001 C CNN
-F 3 "~" H 5900 1750 50  0001 C CNN
-	1    5900 1750
+P 6650 1750
+F 0 "C106" H 6765 1796 50  0000 L CNN
+F 1 "100n" H 6765 1705 50  0000 L CNN
+F 2 "" H 6688 1600 50  0001 C CNN
+F 3 "~" H 6650 1750 50  0001 C CNN
+	1    6650 1750
 	1    0    0    -1
 $EndComp
@@
 L power:GND #PWR0118
 U 1 1 5C77C78E
-P 5900 2000
-F 0 "#PWR0118" H 5900 1750 50  0001 C CNN
-F 1 "GND" H 5905 1827 50  0000 C CNN
-F 2 "" H 5900 2000 50  0001 C CNN
-F 3 "" H 5900 2000 50  0001 C CNN
-	1    5900 2000
-	1    0    0    -1
-$EndComp
-Wire Wire Line
-	5900 1900 5900 2000
-Wire Wire Line
-	5900 1600 5900 1500
-Wire Wire Line
-	5900 1500 5550 1500
+P 6650 2000
+F 0 "#PWR0118" H 6650 1750 50  0001 C CNN
+F 1 "GND" H 6655 1827 50  0000 C CNN
+F 2 "" H 6650 2000 50  0001 C CNN
+F 3 "" H 6650 2000 50  0001 C CNN
+	1    6650 2000
+	1    0    0    -1
+$EndComp
+Wire Wire Line
+	6650 1900 6650 2000
+Wire Wire Line
+	6650 1600 6650 1500
+Wire Wire Line
+	6650 1500 6300 1500
 Text Notes 9250 1050 0    167  ~ 0
 LED
@@
 L power:+3.3V #PWR0134
 U 1 1 5C897DE7
-P 5900 1400
-F 0 "#PWR0134" H 5900 1250 50  0001 C CNN
-F 1 "+3.3V" V 5915 1528 50  0000 L CNN
-F 2 "" H 5900 1400 50  0001 C CNN
-F 3 "" H 5900 1400 50  0001 C CNN
-	1    5900 1400
-	1    0    0    -1
-$EndComp
-Wire Wire Line
-	5900 1400 5900 1500
-Connection ~ 5900 1500
-Wire Wire Line
-	4750 1500 5250 1500
+P 5750 1350
+F 0 "#PWR0134" H 5750 1200 50  0001 C CNN
+F 1 "+3.3V" V 5765 1478 50  0000 L CNN
+F 2 "" H 5750 1350 50  0001 C CNN
+F 3 "" H 5750 1350 50  0001 C CNN
+	1    5750 1350
+	1    0    0    -1
+$EndComp
 Wire Wire Line
 	4350 1500 4750 1500
@@
 Wire Wire Line
 	2350 6350 2350 6450
-$Comp
-L power:+3.3V #PWR0136
-U 1 1 5C8AD182
-P 1400 6500
-F 0 "#PWR0136" H 1400 6350 50  0001 C CNN
-F 1 "+3.3V" V 1415 6628 50  0000 L CNN
-F 2 "" H 1400 6500 50  0001 C CNN
-F 3 "" H 1400 6500 50  0001 C CNN
-	1    1400 6500
-	1    0    0    -1
-$EndComp
 Wire Wire Line
 	1400 6500 1400 6700
@@
 	0    1    1    0
 $EndComp
-Wire Wire Line
-	2000 4400 1850 4400
-Wire Wire Line
-	2000 4600 1850 4600
 Text Label 1800 4400 0    50   ~ 0
 MOSI
@@
 	0    -1   -1   0
 $EndComp
+Wire Wire Line
+	5750 1350 5750 1500
+Wire Wire Line
+	5750 1500 6000 1500
+$Comp
+L power:+3.3V #PWR0136
+U 1 1 5C9C380F
+P 4750 1400
+F 0 "#PWR0136" H 4750 1250 50  0001 C CNN
+F 1 "+3.3V" V 4765 1528 50  0000 L CNN
+F 2 "" H 4750 1400 50  0001 C CNN
+F 3 "" H 4750 1400 50  0001 C CNN
+	1    4750 1400
+	1    0    0    -1
+$EndComp
+Wire Wire Line
+	4750 1400 4750 1500
+Connection ~ 4750 1500
+Wire Wire Line
+	6650 1500 6900 1500
+Connection ~ 6650 1500
+Text Label 6800 1500 0    50   ~ 0
+3.3V_Analog
+Text Label 1400 6550 0    50   ~ 0
+3.3V_Analog
+$Comp
+L power:PWR_FLAG #FLG0101
+U 1 1 5C9CA291
+P 4900 1500
+F 0 "#FLG0101" H 4900 1575 50  0001 C CNN
+F 1 "PWR_FLAG" V 4900 1628 50  0000 L CNN
+F 2 "" H 4900 1500 50  0001 C CNN
+F 3 "~" H 4900 1500 50  0001 C CNN
+	1    4900 1500
+	0    1    1    0
+$EndComp
+Wire Wire Line
+	4900 1500 4750 1500
+$Comp
+L power:GND #PWR0272
+U 1 1 5C9CD4C6
+P 5500 2050
+F 0 "#PWR0272" H 5500 1800 50  0001 C CNN
+F 1 "GND" H 5505 1877 50  0000 C CNN
+F 2 "" H 5500 2050 50  0001 C CNN
+F 3 "" H 5500 2050 50  0001 C CNN
+	1    5500 2050
+	1    0    0    -1
+$EndComp
+$Comp
+L power:PWR_FLAG #FLG0102
+U 1 1 5C9CD526
+P 5500 1900
+F 0 "#FLG0102" H 5500 1975 50  0001 C CNN
+F 1 "PWR_FLAG" H 5500 2074 50  0000 C CNN
+F 2 "" H 5500 1900 50  0001 C CNN
+F 3 "~" H 5500 1900 50  0001 C CNN
+	1    5500 1900
+	1    0    0    -1
+$EndComp
+Wire Wire Line
+	5500 1900 5500 2050
+$Comp
+L power:PWR_FLAG #FLG0103
+U 1 1 5C9D07F4
+P 6650 1350
+F 0 "#FLG0103" H 6650 1425 50  0001 C CNN
+F 1 "PWR_FLAG" H 6650 1524 50  0000 C CNN
+F 2 "" H 6650 1350 50  0001 C CNN
+F 3 "~" H 6650 1350 50  0001 C CNN
+	1    6650 1350
+	1    0    0    -1
+$EndComp
+Wire Wire Line
+	6650 1350 6650 1500
+$Comp
+L power:PWR_FLAG #FLG0104
+U 1 1 5C9D6F94
+P 2900 3400
+F 0 "#FLG0104" H 2900 3475 50  0001 C CNN
+F 1 "PWR_FLAG" H 2900 3574 50  0000 C CNN
+F 2 "" H 2900 3400 50  0001 C CNN
+F 3 "~" H 2900 3400 50  0001 C CNN
+	1    2900 3400
+	1    0    0    -1
+$EndComp
+Wire Wire Line
+	2900 3400 2900 3500
+Connection ~ 2900 3500
+Wire Wire Line
+	2900 3500 2500 3500
+Wire Wire Line
+	1800 4600 2000 4600
+Wire Wire Line
+	2000 4400 1800 4400
 $EndSCHEMATC

Commit message: Update Schema
Footprint
Netlist
Parts:
- C101, C104: footprint (none) -> Capacitor_SMD:CP_Elec_8x6.2
- C102, C103, C105, C106: footprint (none) -> Capacitor_SMD:C_0805_2012Metric
- D101: footprint (none) -> Diode_SMD:D_SMB
- FB101, R101, R102, R103, R104, R105, R106, R107, R108, R109, R110: footprint (none) -> Resistor_SMD:R_0805_2012Metric
- J101: footprint (none) -> Connector_PinSocket_2.54mm:PinSocket_2x20_P2.54mm_Vertical
- L101: footprint (none) -> myFoodprints:SDR1006-470KL
- RV101: footprint (none) -> Potentiometer_THT:Potentiometer_Alps_RK09K_Single_Vertical
- SW101, SW102, SW103, SW104, SW105, SW106: footprint (none) -> myFoodprints:TSA12100TACTSWITCH
- Y101: footprint (none) -> myFoodprints:Piezo CE-C75
Changed lines of the file:
@@
 F 0 "J101" H 2250 5517 50  0000 C CNN
 F 1 "Conn_02x20_Odd_Even" H 2250 5426 50  0000 C CNN
-F 2 "" H 2200 4400 50  0001 C CNN
+F 2 "Connector_PinSocket_2.54mm:PinSocket_2x20_P2.54mm_Vertical" H 2200 4400 50  0001 C CNN
 F 3 "~" H 2200 4400 50  0001 C CNN
 	1    2200 4400
@@
 F 0 "FB101" V 6424 1500 50  0000 C CNN
 F 1 "Ferrite_Bead" V 6333 1500 50  0000 C CNN
-F 2 "" V 6080 1500 50  0001 C CNN
+F 2 "Resistor_SMD:R_0805_2012Metric" V 6080 1500 50  0001 C CNN
 F 3 "~" H 6150 1500 50  0001 C CNN
 	1    6150 1500
@@
 F 0 "C106" H 6765 1796 50  0000 L CNN
 F 1 "100n" H 6765 1705 50  0000 L CNN
-F 2 "" H 6688 1600 50  0001 C CNN
+F 2 "Capacitor_SMD:C_0805_2012Metric" H 6688 1600 50  0001 C CNN
 F 3 "~" H 6650 1750 50  0001 C CNN
 	1    6650 1750
@@
 F 0 "R105" V 5243 4150 50  0000 C CNN
 F 1 "1k" V 5334 4150 50  0000 C CNN
-F 2 "" V 5380 4150 50  0001 C CNN
+F 2 "Resistor_SMD:R_0805_2012Metric" V 5380 4150 50  0001 C CNN
 F 3 "~" H 5450 4150 50  0001 C CNN
 	1    5450 4150
@@
 F 0 "R106" V 5243 4700 50  0000 C CNN
 F 1 "1k" V 5334 4700 50  0000 C CNN
-F 2 "" V 5380 4700 50  0001 C CNN
+F 2 "Resistor_SMD:R_0805_2012Metric" V 5380 4700 50  0001 C CNN
 F 3 "~" H 5450 4700 50  0001 C CNN
 	1    5450 4700
@@
 F 0 "R107" V 5243 5300 50  0000 C CNN
 F 1 "1k" V 5334 5300 50  0000 C CNN
-F 2 "" V 5380 5300 50  0001 C CNN
+F 2 "Resistor_SMD:R_0805_2012Metric" V 5380 5300 50  0001 C CNN
 F 3 "~" H 5450 5300 50  0001 C CNN
 	1    5450 5300
@@
 F 0 "R108" V 5243 5900 50  0000 C CNN
 F 1 "1k" V 5334 5900 50  0000 C CNN
-F 2 "" V 5380 5900 50  0001 C CNN
+F 2 "Resistor_SMD:R_0805_2012Metric" V 5380 5900 50  0001 C CNN
 F 3 "~" H 5450 5900 50  0001 C CNN
 	1    5450 5900
@@
 F 0 "R103" V 5193 6400 50  0000 C CNN
 F 1 "1k" V 5284 6400 50  0000 C CNN
-F 2 "" V 5330 6400 50  0001 C CNN
+F 2 "Resistor_SMD:R_0805_2012Metric" V 5330 6400 50  0001 C CNN
 F 3 "~" H 5400 6400 50  0001 C CNN
 	1    5400 6400
@@
 F 0 "R104" V 5193 6950 50  0000 C CNN
 F 1 "1k" V 5284 6950 50  0000 C CNN
-F 2 "" V 5330 6950 50  0001 C CNN
+F 2 "Resistor_SMD:R_0805_2012Metric" V 5330 6950 50  0001 C CNN
 F 3 "~" H 5400 6950 50  0001 C CNN
 	1    5400 6950
@@
 F 0 "SW103" H 5900 4685 50  0000 C CNN
 F 1 "SW_Push_boxtec" H 5900 4594 50  0000 C CNN
-F 2 "" H 5900 4600 50  0001 C CNN
+F 2 "myFoodprints:TSA12100TACTSWITCH" H 5900 4600 50  0001 C CNN
 F 3 "" H 5900 4600 50  0001 C CNN
 	1    5900 4400
@@
 F 0 "SW104" H 5900 5235 50  0000 C CNN
 F 1 "SW_Push_boxtec" H 5900 5144 50  0000 C CNN
-F 2 "" H 5900 5150 50  0001 C CNN
+F 2 "myFoodprints:TSA12100TACTSWITCH" H 5900 5150 50  0001 C CNN
 F 3 "" H 5900 5150 50  0001 C CNN
 	1    5900 4950
@@
 F 0 "SW105" H 5900 5835 50  0000 C CNN
 F 1 "SW_Push_boxtec" H 5900 5744 50  0000 C CNN
-F 2 "" H 5900 5750 50  0001 C CNN
+F 2 "myFoodprints:TSA12100TACTSWITCH" H 5900 5750 50  0001 C CNN
 F 3 "" H 5900 5750 50  0001 C CNN
 	1    5900 5550
@@
 F 0 "SW106" H 5900 6435 50  0000 C CNN
 F 1 "SW_Push_boxtec" H 5900 6344 50  0000 C CNN
-F 2 "" H 5900 6350 50  0001 C CNN
+F 2 "myFoodprints:TSA12100TACTSWITCH" H 5900 6350 50  0001 C CNN
 F 3 "" H 5900 6350 50  0001 C CNN
 	1    5900 6150
@@
 F 0 "SW101" H 5850 6935 50  0000 C CNN
 F 1 "SW_Push_boxtec" H 5850 6844 50  0000 C CNN
-F 2 "" H 5850 6850 50  0001 C CNN
+F 2 "myFoodprints:TSA12100TACTSWITCH" H 5850 6850 50  0001 C CNN
 F 3 "" H 5850 6850 50  0001 C CNN
 	1    5850 6650
@@
 F 0 "SW102" H 5850 7485 50  0000 C CNN
 F 1 "SW_Push_boxtec" H 5850 7394 50  0000 C CNN
-F 2 "" H 5850 7400 50  0001 C CNN
+F 2 "myFoodprints:TSA12100TACTSWITCH" H 5850 7400 50  0001 C CNN
 F 3 "" H 5850 7400 50  0001 C CNN
 	1    5850 7200
@@
 F 0 "RV101" H 1330 6896 50  0000 R CNN
 F 1 "R_POT_boxtec" H 1330 6805 50  0000 R CNN
-F 2 "" H 1400 6850 50  0001 C CNN
+F 2 "Potentiometer_THT:Potentiometer_Alps_RK09K_Single_Vertical" H 1400 6850 50  0001 C CNN
 F 3 "" H 1400 6850 50  0001 C CNN
 	1    1400 6850
@@
 F 0 "D101" V 3454 1879 50  0000 L CNN
 F 1 "MBRS1100T3G" V 3545 1879 50  0000 L CNN
-F 2 "" H 3500 1800 50  0001 C CNN
+F 2 "Diode_SMD:D_SMB" H 3500 1800 50  0001 C CNN
 F 3 "~" H 3500 1800 50  0001 C CNN
 	1    3500 1800
@@
 F 0 "R101" V 743 3300 50  0000 C CNN
 F 1 "DNP" V 834 3300 50  0000 C CNN
-F 2 "" V 880 3300 50  0001 C CNN
+F 2 "Resistor_SMD:R_0805_2012Metric" V 880 3300 50  0001 C CNN
 F 3 "~" H 950 3300 50  0001 C CNN
 	1    950  3300
@@
 F 0 "R102" V 1093 3300 50  0000 C CNN
 F 1 "DNP" V 1184 3300 50  0000 C CNN
-F 2 "" V 1230 3300 50  0001 C CNN
+F 2 "Resistor_SMD:R_0805_2012Metric" V 1230 3300 50  0001 C CNN
 F 3 "~" H 1300 3300 50  0001 C CNN
 	1    1300 3300
@@
 F 0 "Y101" V 9104 4781 50  0000 L CNN
 F 1 "Piezo_boxtec" V 9195 4781 50  0000 L CNN
-F 2 "" H 9150 4650 50  0001 C CNN
+F 2 "myFoodprints:Piezo CE-C75" H 9150 4650 50  0001 C CNN
 F 3 "" H 9150 4650 50  0001 C CNN
 	1    9150 4650
@@
 F 0 "R110" V 8943 3800 50  0000 C CNN
 F 1 "300" V 9034 3800 50  0000 C CNN
-F 2 "" V 9080 3800 50  0001 C CNN
+F 2 "Resistor_SMD:R_0805_2012Metric" V 9080 3800 50  0001 C CNN
 F 3 "~" H 9150 3800 50  0001 C CNN
 	1    9150 3800
@@
 F 0 "R109" V 8393 4200 50  0000 C CNN
 F 1 "1k" V 8484 4200 50  0000 C CNN
-F 2 "" V 8530 4200 50  0001 C CNN
+F 2 "Resistor_SMD:R_0805_2012Metric" V 8530 4200 50  0001 C CNN
 F 3 "~" H 8600 4200 50  0001 C CNN
 	1    8600 4200
@@
 F 0 "C103" H 3915 6946 50  0000 L CNN
 F 1 "100n" H 3915 6855 50  0000 L CNN
-F 2 "" H 3838 6750 50  0001 C CNN
+F 2 "Capacitor_SMD:C_0805_2012Metric" H 3838 6750 50  0001 C CNN
 F 3 "~" H 3800 6900 50  0001 C CNN
 	1    3800 6900
@@
 F 0 "C105" H 4865 1796 50  0000 L CNN
 F 1 "100n" H 4865 1705 50  0000 L CNN
-F 2 "" H 4788 1600 50  0001 C CNN
+F 2 "Capacitor_SMD:C_0805_2012Metric" H 4788 1600 50  0001 C CNN
 F 3 "~" H 4750 1750 50  0001 C CNN
 	1    4750 1750
@@
 F 0 "C104" H 4468 1796 50  0000 L CNN
 F 1 "100u" H 4468 1705 50  0000 L CNN
-F 2 "" H 4388 1600 50  0001 C CNN
+F 2 "Capacitor_SMD:CP_Elec_8x6.2" H 4388 1600 50  0001 C CNN
 F 3 "~" H 4350 1750 50  0001 C CNN
 	1    4350 1750
@@
 F 0 "C101" H 1068 1596 50  0000 L CNN
 F 1 "100u" H 1068 1505 50  0000 L CNN
-F 2 "" H 988 1400 50  0001 C CNN
+F 2 "Capacitor_SMD:CP_Elec_8x6.2" H 988 1400 50  0001 C CNN
 F 3 "~" H 950 1550 50  0001 C CNN
 	1    950  1550
@@
 F 0 "C102" H 1515 1596 50  0000 L CNN
 F 1 "100n" H 1515 1505 50  0000 L CNN
-F 2 "" H 1438 1400 50  0001 C CNN
+F 2 "Capacitor_SMD:C_0805_2012Metric" H 1438 1400 50  0001 C CNN
 F 3 "~" H 1400 1550 50  0001 C CNN
 	1    1400 1550
@@
 F 0 "L101" V 4040 1500 50  0000 C CNN
 F 1 "68u" V 3949 1500 50  0000 C CNN
-F 2 "" H 3850 1500 50  0001 C CNN
+F 2 "myFoodprints:SDR1006-470KL" H 3850 1500 50  0001 C CNN
 F 3 "~" H 3850 1500 50  0001 C CNN
 	1    3850 1500
